File: pico-eink.kicad_sch (KiCad schematic)
At the start: 56 parts, among them J1 SM04B-SRSS-TB_LF__SN_, U1 Pico, U2 TPS651851RSLR, U3 ED060XC5

Commit message: 1st raw version, no DRM passed
Parts:
- removed C13, C2: 1uF/25V, Capacitor_SMD:C_0805_2012Metric, symbol Device:C
- removed C14: 1uF/50V, Capacitor_SMD:C_1206_3216Metric, symbol Device:C
- removed C15, C17: 10nF, Capacitor_SMD:C_0805_2012Metric, symbol Device:C
- removed C16, C18, C21, C3: 4.7uF, Capacitor_SMD:C_0805_2012Metric, symbol Device:C
- removed C22, C23: 100nF, Capacitor_SMD:C_0805_2012Metric, symbol Device:C
- removed R1: 5K, symbol Device:R
- removed R10, R7: 1M, Resistor_SMD:R_0603_1608Metric, symbol Device:R
- removed R2, R3, R5, R8: 47k, Resistor_SMD:R_0603_1608Metric, symbol Device:R
- removed R4: 100k, Resistor_SMD:R_0603_1608Metric, symbol Device:R
- removed R6: 43k, Resistor_SMD:R_0603_1608Metric, symbol Device:R
- removed R9: 52.3k, Resistor_SMD:R_0603_1608Metric, symbol Device:R
- removed U2: TPS651851RSLR, footprint:TPS651851RSLR, symbol epdiy:TPS651851RSLR
- added C28, C31: 4.7uF, Capacitor_SMD:C_0805_2012Metric, symbol Device:C
- added C29, C30: 100nF, Capacitor_SMD:C_0805_2012Metric, symbol Device:C
- added C32: 10uF, Capacitor_SMD:C_0805_2012Metric, symbol Device:C
- added C33: 2.2uF, Capacitor_SMD:C_0805_2012Metric, symbol Device:C
- added C34, C36: 1uF/50V, Capacitor_SMD:C_1206_3216Metric, symbol Device:C
- added C35, C37, C38: 1uF/25V, Capacitor_SMD:C_0805_2012Metric, symbol Device:C
- added J2: Conn_02x15, Connector_PinHeader_2.54mm:PinHeader_2x15_P2.54mm_Vertical, symbol Connector_Generic:Conn_02x15_Odd_Even
- added R18: 43k, Resistor_SMD:R_0603_1608Metric, symbol Device:R
- added R19, R23: 1M, Resistor_SMD:R_0603_1608Metric, symbol Device:R
- added R20: 52.3k, Resistor_SMD:R_0603_1608Metric, symbol Device:R
- added R24: 47.5k, Resistor_SMD:R_0603_1608Metric, symbol Device:R
- added R26, R27, R28, R29: 47k, Resistor_SMD:R_0603_1608Metric, symbol Device:R
- added R30: 100k, Resistor_SMD:R_0603_1608Metric, symbol Device:R
- added TP6: BOR, TestPoint:TestPoint_Pad_D2.5mm, symbol Connector:TestPoint
- added U3: TPS651851RSLR, footprints:TPS651851RSLR, symbol epdiy:TPS651851RSLR
- C10, C6: value 4.7uF -> 22uF; LCSC C1779 -> C45783
- C11: value 1uF/25V -> 4.7uF; LCSC C28323 -> C1779
- C19: value 2.2uF -> 10uF; LCSC C49217 -> C15850
- C20: value 1uF/50V -> 10nF; footprint Capacitor_SMD:C_1206_3216Metric -> Capacitor_SMD:C_0805_2012Metric; LCSC C1848 -> C1710
- C25: value 10uF -> 10nF; LCSC C15850 -> C1710
- C26: value 2.2uF -> 4.7uF; LCSC C49217 -> C1779
- C27: value 10uF -> 2.2uF; LCSC C15850 -> C49217
- C5: value 22uF -> 4.7uF; LCSC C45783 -> C1779
- C8: value 10uF -> 4.7uF; LCSC C15850 -> C1779
- C9: value 22uF -> 10uF; LCSC C45783 -> C15850
- J1: footprint footprint:QWIIC_SM04B-SRSS-TB_LFSN_ -> footprints:QWIIC_SM04B-SRSS-TB_LFSN_
- R11: value 47.5k -> 5.1k; LCSC C25819 -> C23186
- TP1: value -15V -> +22V
- TP2: value +15V -> -15V
- TP3: value VCOM -> -20V
- TP4: value +22V -> +15V
- TP5: value -20V -> VCOM
- U1: footprint RPi_Pico:RPi_Pico_SMD_TH -> footprints:RPi_Pico_SMD_TH
- U4: renamed from U3; footprint epaper-breakout:X05A20H34G -> footprints:X05A20H34G
Connections:
- net +22V: now also TP1.1, C33.1, C34.1, R23.1, R26.1, U3.35 (VDDH_DIS); no longer C26.1, TP4.1
- net -15V: now also C8.2, TP2.1, C35.1, R27.1, U3.3 (VNEG), U3.9 (VNEG_DIS); no longer C7.2, TP1.1
- net -20V: now also C27.2, TP3.1, C36.1, R19.1, R28.1, U3.29 (VEE_DIS); no longer C19.2, C20.1, TP5.1
- net 15V: now also TP4.1, C31.2, C37.1, R29.1, U3.19 (VPOS_DIS), U3.44 (VPOS); no longer C11.1, C24.2, TP2.1
- net 3.3V: now also U3.45 (VIN3P3)
- net CKV: now also J2.6 (Pin_6)
- net EPD_VDD: now also C19.1, U3.46 (V3P3); no longer C27.1
- net EP_MODE: now also J2.2 (Pin_2)
- net EP_OE: now also J2.8 (Pin_8)
- net EP_STV: now also J2.4 (Pin_4)
- net EP_VCOM: now also C5.2, TP5.1, C38.1, R30.1, U3.15 (VCOM); no longer C4.2, TP3.1
- net GND: now also C11.1, C19.2, C24.2, C26.1, C27.1, C6.1, C7.2, C8.1, C9.2, U1.3 (GND), U1.8 (GND), C28.1, C29.1, C30.2, C31.1, C32.1, C33.2, C34.2, C35.2, C36.2, C37.2, C38.2, R18.1, R20.2, R24.2, R26.2, R27.2, R28.2, R29.2, R30.2, U3.14 (VCOM_DIS), U3.32 (PGND2), U3.41 (PGND1), U3.48 (AGND2), U3.6 (DGND), U3.8 (AGND1); no longer C11.2, C19.1, C20.2, C24.1, C25.1, C26.2, C27.2, C6.2, C7.1, C8.2, C9.1, R11.2
- net LEH: now also J2.12 (Pin_12)
- net SCL: now also U3.17 (SCL)
- net SDA: now also U3.18 (SDA)
- net TPS_PWRUP: now also J2.22 (Pin_22), U3.21 (PWRUP)
- net TPS_PWR_GOOD: now also J2.24 (Pin_24), U3.23 (PWR_GOOD)
- net TPS_VCOM_CTRL: now also J2.20 (Pin_20), U3.12 (VCOM_CTRL)
- net TPS_WAKEUP: now also J2.16 (Pin_16), U3.5 (WAKEUP)
- net TPS_nINT: now also J2.18 (Pin_18), U3.2 (NINT)
- net VNEG_IN: now also C24.1, C7.1, U3.16 (VCOM_PWR), U3.22 (PBKG), U3.26 (VN), U3.27 (VEE_IN), U3.4 (VNEG_IN), U3.49 (EPAD); no longer C6.1
- net XCL: now also J2.10 (Pin_10)
- net XSTL: now also J2.14 (Pin_14)
- net at D2.1 (K): now also C30.1, U3.30 (VEE_D)
- net at D2.2 (A), D3.1 (K): now also C20.1
- net at TH1.1: now also R18.2, U3.47 (TS)
- net at D5.2 (A): now also C29.2, U3.34 (VDDH_D)
- net at R11.1: now also U1.37 (3V3_EN)
- net at D4.2 (A), L2.2: now also U3.40 (VB_SW)
- net at D4.1 (K): now also C26.2, C28.2, U3.37 (VDDH_IN), U3.42 (VB), U3.43 (VPOS_IN)
- net TPS_WAKEUP_A: now reaches U1.1 (GPIO0)
- net TPS_WAKEUP_A: now also J2.15 (Pin_15)
- net EP_MODE_A: now reaches U1.10 (GPIO7)
- net EP_MODE_A: now also J2.1 (Pin_1)
- net EP_STV_A: now reaches U1.11 (GPIO8)
- net EP_STV_A: now also J2.3 (Pin_3)
- net CKV_A: now reaches U1.12 (GPIO9)
- net CKV_A: now also J2.5 (Pin_5)
- net EP_OE_A: now reaches U1.14 (GPIO10)
- net EP_OE_A: now also J2.7 (Pin_7)
- net XCL_A: now reaches U1.15 (GPIO11)
- net XCL_A: now also J2.9 (Pin_9)
- net TPS_nINT_A: now reaches U1.2 (GPIO1)
- net TPS_nINT_A: now also J2.17 (Pin_17)
- net IO20: now reaches U1.26 (GPIO20)
- net IO20: now also J2.25 (Pin_25)
- net XSTL_A: now reaches U1.27 (GPIO21)
- net XSTL_A: now also J2.13 (Pin_13)
- net LEH_A: now reaches U1.29 (GPIO22)
- net LEH_A: now also J2.11 (Pin_11)
- net IO26: now reaches U1.31 (GPIO26_ADC0)
- net IO26: now also J2.27 (Pin_27)
- net IO27: now reaches U1.32 (GPIO27_ADC1)
- net IO27: now also J2.29 (Pin_29)
- net AGND: now reaches U1.33 (AGND)
- net AGND: now also J2.28 (Pin_28)
- net IO28: now reaches U1.34 (GPIO28_ADC2)
- net IO28: now also J2.26 (Pin_26)
- net ADC_VREF: now reaches U1.35 (ADC_VREF)
- net ADC_VREF: now also J2.30 (Pin_30)
- net TPS_VCOM_CTRL_A: now reaches U1.4 (GPIO2)
- net TPS_VCOM_CTRL_A: now also J2.19 (Pin_19)
- net TPS_PWRUP_A: now reaches U1.5 (GPIO3)
- net TPS_PWRUP_A: now also J2.21 (Pin_21)
- net TPS_PWR_GOOD_A: now reaches U1.9 (GPIO6)
- net TPS_PWR_GOOD_A: now also J2.23 (Pin_23)
- net at D1.1 (K), L1.1: now also U3.25 (VN_SW)
- net VIN: now reaches C10.2
- net VIN: now also C12.1, C6.2, C9.1, L2.1, R11.2, U1.40 (VBUS), C32.2, U3.10 (VIN), U3.24 (VIN_P)
- net at D5.1 (K), D6.2 (A): now also C25.1
- removed net 5V: C12.1, C25.2, C5.2, C8.1, C9.2, L2.1, U1.40 (VBUS)
- net BORDER: no longer names the net of U4.31 (BORDER)
- net BORDER: now also TP6.1
- new net: R23.2, R24.1, U3.33 (VDDH_FB)
- new net: C11.2, U3.1 (VREF)
- new net: C20.2, U3.28 (VEE_DRV)
- new net: R19.2, R20.1, U3.31 (VEE_FB)
- new net: C4.2, U3.7 (INT_LDO)
- new net: C25.2, U3.36 (VDDH_DRV)
- no-connect marks 8 -> 9
Other:
- note added: "EP_MODE EP_STV CKV"
- note added: "EP_OE XCL LEH XSTL"
- note added: "TPS_WAKEUP TPS_nINT TPS_VCOM_CTRL TPS_PWRUP TPS_PWRGOOD"
- moved on the sheet: U1
